File: hardware/rp2040-target.kicad_pcb (KiCad board)
At the start: 2 copper layers, 52.5 x 64.5 mm, 17 parts, among them U2 W25Q128JVS, U3 RP2040

Commit message: SCK change
Connections:
- Y1 pad 12: unconnected-(Y1-SCK-Pad12) -> /RP2040/SWCLK
- Y1 pad 17: /RP2040/SWCLK -> unconnected-(Y1-PDIC-Pad17)
Routing:
- net /RP2040/SWCLK: track 33.7 -> 35.1 mm
Changed lines of the file:
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@@
 		)
 		(sheetname "/")
-		(sheetfile "RP2040_target_board.kicad_sch")
+		(sheetfile "rp2040-target.kicad_sch")
 		(units
 			(unit
@@
 			)
 		)
-		(attr smd)
+		(attr smd exclude_from_pos_files exclude_from_bom)
 		(duplicate_pad_numbers_are_jumpers no)
 		(fp_line
@@
 			(layers "*.Cu" "*.Mask")
 			(remove_unused_layers no)
-			(net "unconnected-(Y1-SCK-Pad12)")
+			(net "/RP2040/SWCLK")
 			(pinfunction "SCK_12")
-			(pintype "passive+no_connect")
+			(pintype "passive")
 		)
 		(pad "13" thru_hole circle
@@
 			(layers "*.Cu" "*.Mask")
 			(remove_unused_layers no)
-			(net "/RP2040/SWCLK")
+			(net "unconnected-(Y1-PDIC-Pad17)")
 			(pinfunction "PDIC_17")
-			(pintype "passive")
+			(pintype "passive+no_connect")
 		)
 		(pad "18" thru_hole circle
@@
 	)
 	(gr_text "SWCLK\n"
-		(at 106.125 125.8 0)
+		(at 106.12 113.08 0)
 		(layer "F.SilkS")
 		(effects
@@
 	)
 	(segment
-		(start 119.5 125.8)
-		(end 102 125.8)
+		(start 104.74 113.1)
+		(end 112.797157 121.157157)
+		(width 0.2)
+		(layer "B.Cu")
+		(net "/RP2040/SWCLK")
+	)
+	(segment
+		(start 102 113.1)
+		(end 104.74 113.1)
+		(width 0.2)
+		(layer "B.Cu")
+		(net "/RP2040/SWCLK")
+	)
+	(segment
+		(start 112.797157 121.157157)
+		(end 124.142843 121.157157)
 		(width 0.2)
 		(layer "B.Cu")
@@
 	(segment
 		(start 126.8 118.5)
-		(end 119.5 125.8)
+		(end 126.8 116.9)
 		(width 0.2)
 		(layer "B.Cu")
@@
 	)
 	(segment
-		(start 126.8 116.9)
+		(start 124.142843 121.157157)
 		(end 126.8 118.5)
 		(width 0.2)
