File: hardware/rp2040-target.kicad_sch (KiCad schematic)
At the start: 1 part

Commit message: SCK change
Connections:
- net RP2040/SWCLK: now also Y1.12 (SCK); no longer Y1.17 (PDIC)
Changed lines of the file:
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@@
-	)
-	(no_connect
-		(at 74.93 105.41)
 	)
 	(no_connect
@@
 	)
 	(no_connect
+		(at 72.39 118.11)
+	)
+	(no_connect
 		(at 74.93 123.19)
 	)
@@
 	(wire
 		(pts
+			(xy 78.74 105.41) (xy 78.74 118.11)
+		)
+		(stroke
+			(width 0)
+			(type default)
+		)
+	)
+	(wire
+		(pts
 			(xy 189.23 88.9) (xy 196.85 88.9)
 		)
@@
 	(wire
 		(pts
-			(xy 72.39 105.41) (xy 74.93 105.41)
+			(xy 72.39 105.41) (xy 78.74 105.41)
 		)
 		(stroke
@@
 	(wire
 		(pts
-			(xy 72.39 118.11) (xy 83.82 118.11)
+			(xy 78.74 118.11) (xy 83.82 118.11)
 		)
 		(stroke
@@
 		)
 		(instances
-			(project "RP2040_target_board"
+			(project "rp2040-target"
 				(path "/061c03c6-5564-4c47-a1f4-f453d6b6ec2c"
 					(reference "#PWR023")
@@
 		)
 		(instances
-			(project "RP2040_target_board"
+			(project "rp2040-target"
 				(path "/061c03c6-5564-4c47-a1f4-f453d6b6ec2c"
 					(reference "#PWR026")
@@
 		)
 		(instances
-			(project "RP2040_target_board"
+			(project "rp2040-target"
 				(path "/061c03c6-5564-4c47-a1f4-f453d6b6ec2c"
 					(reference "#PWR020")
@@
 		)
 		(instances
-			(project "RP2040_target_board"
+			(project "rp2040-target"
 				(path "/061c03c6-5564-4c47-a1f4-f453d6b6ec2c"
 					(reference "#PWR029")
@@
 		)
 		(instances
-			(project "RP2040_target_board"
+			(project "rp2040-target"
 				(path "/061c03c6-5564-4c47-a1f4-f453d6b6ec2c"
 					(reference "#PWR018")
@@
 		)
 		(instances
-			(project "RP2040_target_board"
+			(project "rp2040-target"
 				(path "/061c03c6-5564-4c47-a1f4-f453d6b6ec2c"
 					(reference "#PWR028")
@@
 		)
 		(instances
-			(project "RP2040_target_board"
+			(project "rp2040-target"
 				(path "/061c03c6-5564-4c47-a1f4-f453d6b6ec2c"
 					(reference "#PWR027")
@@
 		)
 		(instances
-			(project "RP2040_target_board"
+			(project "rp2040-target"
 				(path "/061c03c6-5564-4c47-a1f4-f453d6b6ec2c"
 					(reference "#PWR022")
@@
 		)
 		(instances
-			(project "RP2040_target_board"
+			(project "rp2040-target"
 				(path "/061c03c6-5564-4c47-a1f4-f453d6b6ec2c"
 					(reference "#PWR019")
@@
 		)
 		(instances
-			(project "RP2040_target_board"
+			(project "rp2040-target"
 				(path "/061c03c6-5564-4c47-a1f4-f453d6b6ec2c"
 					(reference "#PWR025")
@@
 		)
 		(instances
-			(project "RP2040_target_board"
+			(project "rp2040-target"
 				(path "/061c03c6-5564-4c47-a1f4-f453d6b6ec2c"
 					(reference "Y1")
@@
 		)
 		(instances
-			(project "RP2040_target_board"
+			(project "rp2040-target"
 				(path "/061c03c6-5564-4c47-a1f4-f453d6b6ec2c"
 					(reference "#PWR021")
@@
 		)
 		(instances
-			(project "RP2040_target_board"
+			(project "rp2040-target"
 				(path "/061c03c6-5564-4c47-a1f4-f453d6b6ec2c"
 					(reference "#PWR024")
@@
 		)
 		(instances
-			(project "RP2040_target_board"
+			(project "rp2040-target"
 				(path "/061c03c6-5564-4c47-a1f4-f453d6b6ec2c"
 					(page "2")
@@
 		)
 		(instances
-			(project "RP2040_target_board"
+			(project "rp2040-target"
 				(path "/061c03c6-5564-4c47-a1f4-f453d6b6ec2c"
 					(page "3")
